File: bluetooth_bma400.brd (EAGLE design)
At the start: 38.1 x 38.1 mm, 20 parts, among them IC1 BLUENRG-M2SP, J2 455-1750-1-ND, U1 BMA400

Commit message: Updated files
Parts:
- removed BT1: BU2032SM-JJ-GTR, BU2032SM-JJ-GTR:BAT_BU2032SM-JJ-GTR
- removed C4: 10nF, SparkFun-Capacitors:0603
- removed INT1, TP2: TPB1,27, testpad:B1,27
- removed R4, R5: 2.2k, SparkFun-Resistors:0603
- removed S2: (no value), SparkFun-Switches:SWITCH_SPST_SMD_A
- removed U1: BMA400, BMA400:XDCR_BMA400
- moved J1 28.7 mm to (-15.3, 0.10), turned to 270 degrees
- moved J2 25.6 mm to (-10.2, -4.67)
- moved C2 20.7 mm to (8.74, 3.86)
- moved IC1 16.0 mm to (-1.09, 14.1), turned to 0 degrees
- moved R3 13.7 mm to (-1.80, 23.0)
- moved J3 12.8 mm to (-1.14, 26.1)
- moved R2 12.0 mm to (6.99, 1.78)
- moved C3 10.2 mm to (4.78, 5.44)
- moved D1 9.25 mm to (13.0, -5.87)
- moved S1 6.84 mm to (-1.35, 1.68)
- moved C1 6.35 mm to (-9.42, 3.35)
- moved R1 6.35 mm to (11.5, -0.91)
Connections:
- removed net INT2: TP2.TP, U1.6
- removed net N$2: BT1.+, S2.2
- net GND: no longer BT1.-, C4.1, U1.1, U1.8, U1.9
- net INT1: no longer INT1.TP, U1.5
- net SCL: no longer R4.1, U1.12
- net SDA: no longer R5.1, U1.2
- net VIN: no longer C4.2, R4.2, R5.2, S2.3, U1.10, U1.3, U1.7
Routing:
- net VIN: track 93.4 -> 0.00 mm, vias 9 -> 0
- net SCL: track 56.4 -> 0.00 mm, vias 2 -> 0
- net SDA: track 43.4 -> 0.00 mm, vias 2 -> 0
- net RST: track 30.5 -> 0.00 mm
- net RX: track 28.2 -> 0.00 mm, vias 1 -> 0
- net INT1: track 25.9 -> 0.00 mm
- net TX: track 25.4 -> 0.00 mm, vias 1 -> 0
- net SWCLK: track 22.4 -> 0.00 mm
- net SWDIO: track 19.1 -> 0.00 mm
- net N$2: track 12.5 -> 0.00 mm
- net BOOT: track 10.6 -> 0.00 mm
- net TEST: track 6.88 -> 0.00 mm
- net INT2: track 6.19 -> 0.00 mm
- net N$1: track 1.76 -> 0.00 mm
Other:
- board size 38.1 x 38.1 mm -> 74.3 x 73.2 mm
- board text removed: "03-01-2021"
- board text removed: "CLK"
- board text removed: "DIO"
- board text removed: "GND"
- board text removed: "Low Cost Pedometer"
- board text removed: "RST"
- board text removed: "RX"
- board text removed: "TX"
- board text removed: "VIN"

Commit message: PCB design + library check-in
Parts:
- removed C1: 10nF, SparkFun-Capacitors:0603
- removed C3: 15pF, SparkFun-Capacitors:0603
- removed R1: 10k, SparkFun-Resistors:0603
- removed R3: 47k, SparkFun-Resistors:0603
- removed S1: MOMENTARY-SWITCH-SPST-SMD-4.6X2.8MM, SparkFun-Switches:TACTILE_SWITCH_SMD_4.6X2.8MM
Connections:
- net BOOT: no longer C3.1, R1.2, S1.1, S1.2
- net GND: no longer C1.2, C3.2, R1.1
- net RST: no longer C1.1, R3.1
- net VIN: no longer R3.2, S1.3, S1.4

Commit message: Final version
Parts:
- removed J2: 455-1750-1-ND, SparkFun-Connectors:1X03
- added C1, C3: 0.1uF, SparkFun-Capacitors:0603
- added J4: (no value), SparkFun-Connectors:1X04_SMD_RA_MALE
- added R1, R3: 2.2k, SparkFun-Resistors:0603
- added SW1: REVERSE_SWITCH, reverse_mount_sw:REVERSE_TACTILE
- added U1: BME680, BME680:PSON80P300X300X100-8N
- added U2: LSM6DSO32TRLGA-14L_2P5X3X0P83_STM-M, LSM6DSO32:LGA-14L_2P5X3X0P83_STM-M
- J1: value (none) -> CORTEX_DEBUG_SMD; device SparkFun-Connectors:1X05 -> SparkFun-Connectors:SAMTECH_FTSH-105-01
- J3: value (none) -> QWIIC; device SparkFun-Connectors:1X04_1MM_RA -> BM04B-SRSS-TB_LF__SN_:CONN_BM04B-SRSS-TB(LF)(SN)
- moved D1 27.7 mm to (-8.23, 12.0), turned to 180 degrees
- moved C2 24.6 mm to (-11.3, 18.1)
- moved J1 23.9 mm to (5.08, 12.7), turned to 0 degrees
- moved R2 19.8 mm to (-7.32, 15.5), turned to 270 degrees
- moved J3 13.6 mm to (-2.36, 12.6)
- moved IC1 9.90 mm to (-2.01, 24.0)
Connections:
- removed net BOOT: IC1.7
- removed net RST: IC1.19, J1.5
- new net BUTTON: IC1.7, SW1.P$1, SW1.P$2
- new net INT2: IC1.17, U2.9
- new net NRST: IC1.19, J1.10
- net GND: now also C1.1, C3.2, J1.5, J3.S1, J3.S2, J4.3, SW1.P$3, SW1.P$4, U1.1, U1.5, U1.7, U2.1, U2.6, U2.7; no longer J2.3
- net INT1: now also IC1.18, U2.4; no longer IC1.20
- net RX: now also J4.2; no longer J2.2
- net SCL: now also R3.1, U1.4, U2.13
- net SDA: now also R1.1, U1.3, U2.14
- net SWCLK: now also J1.4; no longer J1.2
- net SWDIO: now also J1.2; no longer J1.4
- net TX: now also J4.1; no longer J2.1
- net VIN: now also C1.2, C3.1, J4.4, R1.2, R3.2, U1.2, U1.6, U1.8, U2.12, U2.5, U2.8
Routing:
- net VIN: track 0.00 -> 103.6 mm, vias 0 -> 6
- net SCL: track 0.00 -> 53.1 mm, vias 0 -> 2
- net SDA: track 0.00 -> 52.6 mm, vias 0 -> 5
- net BUTTON: track 0.00 -> 39.8 mm
- net INT1: track 0.00 -> 34.0 mm, vias 0 -> 2
- net TX: track 0.00 -> 29.6 mm, vias 0 -> 2
- net INT2: track 0.00 -> 25.8 mm, vias 0 -> 2
- net RX: track 0.00 -> 20.6 mm, vias 0 -> 2
- net NRST: track 0.00 -> 18.1 mm, vias 0 -> 2
- net SWCLK: track 0.00 -> 9.42 mm
- net SWDIO: track 0.00 -> 4.63 mm
- net GND: track 0.00 -> 4.15 mm, vias 0 -> 4
- net TEST: track 0.00 -> 2.76 mm
- net N$1: track 0.00 -> 2.75 mm
