File: bluetooth_bma400.sch (EAGLE design)
At the start: 20 parts, among them IC1 BLUENRG-M2SP, J2 455-1750-1-ND, U1 BMA400

Commit message: Updated files
Parts:
- removed BT1: BU2032SM-JJ-GTR, BU2032SM-JJ-GTR:BU2032SM-JJ-GTR
- removed C4: 10nF, SparkFun-Capacitors:10NF-0603-50V-10%
- removed INT1, TP2: TPB1,27, testpad:TPB1,27
- removed R4, R5: 2.2k, SparkFun-Resistors:2.2KOHM-0603-1/10W-1%
- removed S2: (no value), SparkFun-Switches:SWITCH-SPDT-SMD-RIGHT-ANGLE
- removed U1: BMA400, BMA400:BMA400
Connections:
- removed net INT2: TP2.TP, U1.INT2
- removed net N$2: BT1.+, S2.P
- net GND: no longer BT1.-, C4.1, U1.GND, U1.GNDIO, U1.SDO
- net INT1: no longer INT1.TP, U1.INT1
- net SCL: no longer R4.1, U1.SCX
- net SDA: no longer R5.1, U1.SDX
- net VIN: no longer C4.2, R4.2, R5.2, S2.S, U1.!CSB, U1.VDD, U1.VDDIO

Commit message: PCB design + library check-in
Parts:
- removed C1: 10nF, SparkFun-Capacitors:10NF-0603-50V-10%
- removed C3: 15pF, SparkFun-Capacitors:15PF-0603-50V-5%
- removed R1: 10k, SparkFun-Resistors:10KOHM-0603-1/10W-1%
- removed R3: 47k, SparkFun-Resistors:47KOHM-0603-1/10W-1%
- removed S1: MOMENTARY-SWITCH-SPST-SMD-4.6X2.8MM, SparkFun-Switches:MOMENTARY-SWITCH-SPST-SMD-4.6X2.8MM
Connections:
- net BOOT: no longer C3.1, R1.2, S1.1
- net GND: no longer C1.2, C3.2, R1.1
- net RST: no longer C1.1, R3.1
- net VIN: no longer R3.2, S1.2

Commit message: Final version
Parts:
- removed J2: 455-1750-1-ND, SparkFun-Connectors:CONN_03
- added C1, C3: 0.1uF, SparkFun-Capacitors:0.1UF-0603-25V-(+80/-20%)
- added J4: (no value), SparkFun-Connectors:CONN_04SMD
- added R1, R3: 2.2k, SparkFun-Resistors:2.2KOHM-0603-1/10W-1%
- added SW1: REVERSE_SWITCH, reverse_mount_sw:REVERSE_SWITCH
- added U1: BME680, BME680:BME680
- added U2: LSM6DSO32TRLGA-14L_2P5X3X0P83_STM-M, LSM6DSO32:LSM6DSO32TRLGA-14L_2P5X3X0P83_STM-M
- J1: value (none) -> CORTEX_DEBUG_SMD; device SparkFun-Connectors:CONN_05 -> SparkFun-Connectors:CORTEX_DEBUG_SMD
- J3: value (none) -> QWIIC; device SparkFun-Connectors:QWIIC_CONNECTORJS-1MM -> BM04B-SRSS-TB_LF__SN_:QWIIC
Connections:
- removed net BOOT: IC1.DIO7/BOOT
- removed net RST: IC1.RESETN, J1.5
- new net BUTTON: IC1.DIO7/BOOT, SW1.1, SW1.2
- new net INT2: IC1.DIO3, U2.INT2
- new net NRST: IC1.RESETN, J1.!RESET
- net GND: now also C1.1, C3.2, J1.GND@3, J1.GND@5, J3.P$2, J4.SDA, SW1.3, SW1.4, U1.GND, U1.SDO, U2.GND, U2.GND_2, U2.SDO/SA0; no longer J1.3, J2.3
- net INT1: now also IC1.DIO1, U2.INT1; no longer IC1.DIO12
- net RX: now also J4.SCL; no longer J2.2
- net SCL: now also R3.1, U1.SCK, U2.SCL
- net SDA: now also R1.1, U1.SDI, U2.SDA
- net SWCLK: now also J1.SWDCLK/TCK; no longer J1.2
- net SWDIO: now also J1.SWDIO/TMS; no longer J1.4
- net TX: now also J4.VCC; no longer J2.1
- net VIN: now also C1.2, C3.1, J1.VCC, J4.GND, R1.2, R3.2, U1.CSB, U1.VDD, U1.VDDIO, U2.CS, U2.VDD, U2.VDDIO; no longer J1.1
Other:
- moved on the sheet: C2, D1, R2
