File: hardware/v3/BT40_v23.sch (EAGLE design)
At the start: 14 parts, among them IC1 BLUENRG-M2SP, J1 CORTEX_DEBUG_SMD, J3 QWIIC, SW1 REVERSE_SWITCH, U1 BME680, U2 LSM6DSO32TRLGA-14L_2P5X3X0P83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

Commit message: Changes to design files
Parts:
- added U$1: BM40-B_1, BT40E-lib-11:BM40-B_1
- added U3: BT40F, BT40F:BT40F
Connections:
- new net N$2: U3.SWDCLK
- net GND: now also U3.GND, U3.VSS
Changed lines of the file:
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@@
 <part name="SW1" library="reverse_mount_sw" deviceset="REVERSE_SWITCH" device=""/>
 <part name="GND9" library="Adafruit nRF52 Bluefruit Feather rev G" deviceset="SUPPLY1_GND" device="" value="GND"/>
+<part name="U$1" library="BT40E-lib-11" deviceset="BM40-B_1" device=""/>
+<part name="U3" library="BT40F" deviceset="BT40F" device=""/>
+<part name="GND10" library="Adafruit nRF52 Bluefruit Feather rev G" deviceset="SUPPLY1_GND" device="" value="GND"/>
 </parts>
 <sheets>
@@
 <instance part="GND9" gate="1" x="106.68" y="86.36" smashed="yes">
 <attribute name="VALUE" x="105.156" y="84.836" size="1.016" layer="96" font="vector" ratio="20"/>
+</instance>
+<instance part="U3" gate="G$1" x="-88.9" y="106.68" smashed="yes">
+<attribute name="NAME" x="-109.22" y="158.369" size="1.778" layer="95"/>
+<attribute name="VALUE" x="-109.22" y="53.34" size="1.778" layer="96" font="vector" ratio="20"/>
+</instance>
+<instance part="GND10" gate="1" x="-50.8" y="48.26" smashed="yes">
+<attribute name="VALUE" x="-52.324" y="46.736" size="1.016" layer="96" font="vector" ratio="20"/>
 </instance>
 </instances>
@@
 <wire x1="101.6" y1="93.98" x2="106.68" y2="93.98" width="0.1524" layer="91"/>
 <junction x="106.68" y="93.98"/>
+</segment>
+<segment>
+<pinref part="U3" gate="G$1" pin="VSS"/>
+<pinref part="GND10" gate="1" pin="GND"/>
+<wire x1="-63.5" y1="60.96" x2="-50.8" y2="60.96" width="0.1524" layer="91"/>
+<wire x1="-50.8" y1="60.96" x2="-50.8" y2="58.42" width="0.1524" layer="91"/>
+<pinref part="U3" gate="G$1" pin="GND"/>
+<wire x1="-50.8" y1="58.42" x2="-50.8" y2="50.8" width="0.1524" layer="91"/>
+<wire x1="-63.5" y1="58.42" x2="-50.8" y2="58.42" width="0.1524" layer="91"/>
+<junction x="-50.8" y="58.42"/>
 </segment>
 </net>
@@
 </segment>
 </net>
+<net name="N$2" class="0">
+<segment>
+<pinref part="U3" gate="G$1" pin="SWDCLK"/>
+<wire x1="-114.3" y1="139.7" x2="-121.92" y2="139.7" width="0.1524" layer="91"/>
+</segment>
+</net>

Commit message: Check-in
Connections:
- removed net N$2: U3.SWDCLK
- net SWCLK: now also U3.SWDCLK
Changed lines of the file:
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@@
 <label x="73.66" y="38.1" size="1.016" layer="95" font="vector" ratio="20" xref="yes"/>
+</segment>
+<segment>
+<pinref part="U3" gate="G$1" pin="SWDCLK"/>
+<wire x1="-114.3" y1="139.7" x2="-121.92" y2="139.7" width="0.1524" layer="91"/>
+<label x="-121.92" y="139.7" size="1.778" layer="95" font="vector" ratio="20" rot="R180" xref="yes"/>
 </segment>
 </net>
@@
 </segment>
 </net>
-<net name="N$2" class="0">
-<segment>
-<pinref part="U3" gate="G$1" pin="SWDCLK"/>
-<wire x1="-114.3" y1="139.7" x2="-121.92" y2="139.7" width="0.1524" layer="91"/>
-</segment>
-</net>

Commit message: Changes
Parts:
- removed U$1: BM40-B_1, BT40E-lib-11:BM40-B_1
- added C4: 0.1uF, SparkFun-Capacitors:0.1UF-0603-25V-(+80/-20%)
Connections:
- net GND: now also C4.2
- net NRST: now also U3.!RESET
- net SWDIO: now also U3.SWDIO
- net VIN: now also C4.1, U3.VDDH
Changed lines of the file:
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@@
 <part name="SW1" library="reverse_mount_sw" deviceset="REVERSE_SWITCH" device=""/>
 <part name="GND9" library="Adafruit nRF52 Bluefruit Feather rev G" deviceset="SUPPLY1_GND" device="" value="GND"/>
-<part name="U$1" library="BT40E-lib-11" deviceset="BM40-B_1" device=""/>
 <part name="U3" library="BT40F" deviceset="BT40F" device=""/>
 <part name="GND10" library="Adafruit nRF52 Bluefruit Feather rev G" deviceset="SUPPLY1_GND" device="" value="GND"/>
+<part name="SUPPLY7" library="SparkFun-PowerSymbols" library_urn="urn:adsk.eagle:library:530" deviceset="VIN" device=""/>
+<part name="C4" library="SparkFun-Capacitors" library_urn="urn:adsk.eagle:library:510" deviceset="0.1UF" device="-0603-25V-(+80/-20%)" package3d_urn="urn:adsk.eagle:package:37414/1" value="0.1uF"/>
+<part name="GND11" library="Adafruit nRF52 Bluefruit Feather rev G" deviceset="SUPPLY1_GND" device="" value="GND"/>
 </parts>
 <sheets>
@@
 <instance part="GND10" gate="1" x="-50.8" y="48.26" smashed="yes">
 <attribute name="VALUE" x="-52.324" y="46.736" size="1.016" layer="96" font="vector" ratio="20"/>
+</instance>
+<instance part="SUPPLY7" gate="G$1" x="-43.18" y="160.02" smashed="yes">
+<attribute name="VALUE" x="-43.18" y="162.814" size="1.016" layer="96" font="vector" ratio="20" align="bottom-center"/>
+</instance>
+<instance part="C4" gate="G$1" x="-43.18" y="139.7" smashed="yes">
+<attribute name="NAME" x="-45.466" y="142.621" size="1.016" layer="95" font="vector" ratio="20"/>
+<attribute name="VALUE" x="-47.244" y="138.811" size="1.016" layer="96" font="vector" ratio="20"/>
+</instance>
+<instance part="GND11" gate="1" x="-43.18" y="127" smashed="yes">
+<attribute name="VALUE" x="-44.704" y="125.476" size="1.016" layer="96" font="vector" ratio="20"/>
 </instance>
 </instances>
@@
 <wire x1="-63.5" y1="58.42" x2="-50.8" y2="58.42" width="0.1524" layer="91"/>
 <junction x="-50.8" y="58.42"/>
+</segment>
+<segment>
+<pinref part="C4" gate="G$1" pin="2"/>
+<pinref part="GND11" gate="1" pin="GND"/>
+<wire x1="-43.18" y1="137.16" x2="-43.18" y2="129.54" width="0.1524" layer="91"/>
 </segment>
 </net>
@@
 <junction x="241.3" y="129.032"/>
 </segment>
+<segment>
+<pinref part="SUPPLY7" gate="G$1" pin="VIN"/>
+<wire x1="-43.18" y1="144.78" x2="-43.18" y2="149.86" width="0.1524" layer="91"/>
+<pinref part="C4" gate="G$1" pin="1"/>
+<pinref part="U3" gate="G$1" pin="VDDH"/>
+<wire x1="-43.18" y1="149.86" x2="-43.18" y2="160.02" width="0.1524" layer="91"/>
+<wire x1="-63.5" y1="149.86" x2="-43.18" y2="149.86" width="0.1524" layer="91"/>
+<junction x="-43.18" y="149.86"/>
+</segment>
 </net>
 <net name="SDA" class="0">
@@
 <pinref part="U3" gate="G$1" pin="SWDCLK"/>
 <wire x1="-114.3" y1="139.7" x2="-121.92" y2="139.7" width="0.1524" layer="91"/>
-<label x="-121.92" y="139.7" size="1.778" layer="95" font="vector" ratio="20" rot="R180" xref="yes"/>
+<label x="-121.92" y="139.7" size="1.016" layer="95" font="vector" ratio="20" rot="R180" xref="yes"/>
 </segment>
 </net>
@@
 <label x="73.66" y="40.64" size="1.016" layer="95" font="vector" ratio="20" xref="yes"/>
 </segment>
+<segment>
+<pinref part="U3" gate="G$1" pin="SWDIO"/>
+<wire x1="-114.3" y1="137.16" x2="-121.92" y2="137.16" width="0.1524" layer="91"/>
+<label x="-121.92" y="137.16" size="1.016" layer="95" font="vector" ratio="20" rot="R180" xref="yes"/>
+</segment>
 </net>
 <net name="TX" class="0">
@@
 <label x="73.66" y="30.48" size="1.016" layer="95" font="vector" ratio="20" xref="yes"/>
 </segment>
-</net>
+<segment>
+<pinref part="U3" gate="G$1" pin="!RESET"/>
+<wire x1="-114.3" y1="144.78" x2="-121.92" y2="144.78" width="0.1524" layer="91"/>
+<label x="-121.92" y="144.78" size="1.016" layer="95" font="vector" ratio="20" rot="R180" xref="yes"/>
+</segment>
+</net>

Commit message: Update to schematic
Connections:
- new net 3.3V: U3.VDD
- new net SWO: J1.SWO/TDO, U3.P0.11
- net GND: now also J1.GNDDTCT
- net RX: now also U3.P0.22
- net SCL: now also U3.P1.03
- net SDA: now also U3.P1.02
- net TX: now also U3.P0.20
Changed lines of the file:
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@@
 <part name="C4" library="SparkFun-Capacitors" library_urn="urn:adsk.eagle:library:510" deviceset="0.1UF" device="-0603-25V-(+80/-20%)" package3d_urn="urn:adsk.eagle:package:37414/1" value="0.1uF"/>
 <part name="GND11" library="Adafruit nRF52 Bluefruit Feather rev G" deviceset="SUPPLY1_GND" device="" value="GND"/>
+<part name="SUPPLY8" library="SparkFun-PowerSymbols" library_urn="urn:adsk.eagle:library:530" deviceset="3.3V" device=""/>
 </parts>
 <sheets>
@@
 <attribute name="VALUE" x="-44.704" y="125.476" size="1.016" layer="96" font="vector" ratio="20"/>
 </instance>
+<instance part="SUPPLY8" gate="G$1" x="-50.8" y="160.02" smashed="yes">
+<attribute name="VALUE" x="-50.8" y="162.814" size="1.016" layer="96" font="vector" ratio="20" align="bottom-center"/>
+</instance>
 </instances>
 <busses>
@@
 <pinref part="GND2" gate="1" pin="GND"/>
 <wire x1="35.56" y1="35.56" x2="25.4" y2="35.56" width="0.1524" layer="91"/>
-<wire x1="25.4" y1="35.56" x2="25.4" y2="24.13" width="0.1524" layer="91"/>
+<wire x1="25.4" y1="35.56" x2="25.4" y2="30.48" width="0.1524" layer="91"/>
 <pinref part="J1" gate="G$1" pin="GND@3"/>
+<wire x1="25.4" y1="30.48" x2="25.4" y2="24.13" width="0.1524" layer="91"/>
 <wire x1="35.56" y1="38.1" x2="25.4" y2="38.1" width="0.1524" layer="91"/>
 <wire x1="25.4" y1="38.1" x2="25.4" y2="35.56" width="0.1524" layer="91"/>
 <junction x="25.4" y="35.56"/>
+<pinref part="J1" gate="G$1" pin="GNDDTCT"/>
+<wire x1="35.56" y1="30.48" x2="25.4" y2="30.48" width="0.1524" layer="91"/>
+<junction x="25.4" y="30.48"/>
 </segment>
 <segment>
@@
 <wire x1="228.6" y1="116.84" x2="233.68" y2="116.84" width="0.1524" layer="91"/>
 <label x="233.68" y="116.84" size="1.016" layer="95" font="vector" ratio="20" xref="yes"/>
+</segment>
+<segment>
+<pinref part="U3" gate="G$1" pin="P1.03"/>
+<wire x1="-63.5" y1="111.76" x2="-55.88" y2="111.76" width="0.1524" layer="91"/>
+<label x="-55.88" y="111.76" size="1.016" layer="95" font="vector" ratio="20" xref="yes"/>
 </segment>
 </net>
@@
 <label x="233.68" y="119.38" size="1.016" layer="95" font="vector" ratio="20" xref="yes"/>
 </segment>
+<segment>
+<pinref part="U3" gate="G$1" pin="P1.02"/>
+<wire x1="-63.5" y1="114.3" x2="-55.88" y2="114.3" width="0.1524" layer="91"/>
+<label x="-55.88" y="114.3" size="1.016" layer="95" font="vector" ratio="20" xref="yes"/>
+</segment>
 </net>
 <net name="TEST" class="0">
@@
 <label x="111.76" y="30.48" size="1.016" layer="95" font="vector" ratio="20" xref="yes"/>
 </segment>
+<segment>
+<pinref part="U3" gate="G$1" pin="P0.20"/>
+<wire x1="-63.5" y1="137.16" x2="-58.42" y2="137.16" width="0.1524" layer="91"/>
+<label x="-58.42" y="137.16" size="1.016" layer="95" font="vector" ratio="20" xref="yes"/>
+</segment>
 </net>
 <net name="RX" class="0">
@@
 <wire x1="101.6" y1="33.02" x2="111.76" y2="33.02" width="0.1524" layer="91"/>
 <label x="111.76" y="33.02" size="1.016" layer="95" font="vector" ratio="20" xref="yes"/>
+</segment>
+<segment>
+<pinref part="U3" gate="G$1" pin="P0.22"/>
+<wire x1="-63.5" y1="134.62" x2="-58.42" y2="134.62" width="0.1524" layer="91"/>
+<label x="-58.42" y="134.62" size="1.016" layer="95" font="vector" ratio="20" xref="yes"/>
 </segment>
 </net>
@@
 </segment>
 </net>
+<net name="3.3V" class="0">
+<segment>
+<pinref part="U3" gate="G$1" pin="VDD"/>
+<pinref part="SUPPLY8" gate="G$1" pin="3.3V"/>
+<wire x1="-63.5" y1="152.4" x2="-50.8" y2="152.4" width="0.1524" layer="91"/>
+<wire x1="-50.8" y1="152.4" x2="-50.8" y2="160.02" width="0.1524" layer="91"/>
+</segment>
+</net>
+<net name="SWO" class="0">
+<segment>
+<pinref part="J1" gate="G$1" pin="SWO/TDO"/>
+<wire x1="68.58" y1="35.56" x2="73.66" y2="35.56" width="0.1524" layer="91"/>
+<label x="73.66" y="35.56" size="1.016" layer="95" font="vector" ratio="20" xref="yes"/>
+</segment>
+<segment>
+<pinref part="U3" gate="G$1" pin="P0.11"/>
+<wire x1="-63.5" y1="144.78" x2="-58.42" y2="144.78" width="0.1524" layer="91"/>
+<label x="-58.42" y="144.78" size="1.016" layer="95" font="vector" ratio="20" xref="yes"/>
+</segment>
+</net>

Commit message: Check-in
Parts:
- removed C2: 0.1uF, SparkFun-Capacitors:0.1UF-0603-25V-(+80/-20%)
- removed IC1: BLUENRG-M2SP, SamacSys_Parts:BLUENRG-M2SP
Connections:
- net BUTTON: now also U3.P1.15; no longer IC1.DIO7/BOOT
- net GND: no longer C2.2, IC1.GND
- net INT1: now also U3.P1.08; no longer IC1.DIO1
- net INT2: now also U3.P0.13/IO0; no longer IC1.DIO3
- net NRST: no longer IC1.RESETN
- net RX: no longer IC1.DIO11
- net SCL: no longer IC1.DIO4
- net SDA: no longer IC1.DIO5
- net SWCLK: no longer IC1.DIO9
- net SWDIO: no longer IC1.DIO10
- net TEST: now also U3.P0.30; no longer IC1.ANATEST0/DIO14
- net TX: no longer IC1.DIO8
- net VIN: no longer C2.1, IC1.VIN
Changed lines of the file:
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@@
 <parts>
 <part name="FRAME1" library="frames" library_urn="urn:adsk.eagle:library:229" deviceset="A4L-LOC" device=""/>
-<part name="GND" library="Adafruit nRF52 Bluefruit Feather rev G" deviceset="SUPPLY1_GND" device="" value="GND"/>
-<part name="IC1" library="SamacSys_Parts" deviceset="BLUENRG-M2SP" device=""/>
-<part name="SUPPLY1" library="SparkFun-PowerSymbols" library_urn="urn:adsk.eagle:library:530" deviceset="VIN" device=""/>
-<part name="C2" library="SparkFun-Capacitors" library_urn="urn:adsk.eagle:library:510" deviceset="0.1UF" device="-0603-25V-(+80/-20%)" package3d_urn="urn:adsk.eagle:package:37414/1" value="0.1uF"/>
 <part name="R2" library="SparkFun-Resistors" library_urn="urn:adsk.eagle:library:532" deviceset="8.2KOHM" device="-0603-1/10W-5%" package3d_urn="urn:adsk.eagle:package:39650/1" value="820">
 <attribute name="SPICEPREFIX" value="R"/>
@@
 <attribute name="SHEET" x="230.505" y="5.08" size="2.54" layer="94"/>
 </instance>
-<instance part="GND" gate="1" x="15.24" y="86.36" smashed="yes">
-<attribute name="VALUE" x="13.716" y="84.836" size="1.016" layer="96" font="vector" ratio="20"/>
-</instance>
-<instance part="IC1" gate="G$1" x="38.1" y="134.62" smashed="yes">
-<attribute name="NAME" x="43.434" y="138.176" size="1.016" layer="95" font="vector" ratio="20" align="center-left"/>
-<attribute name="VALUE" x="67.31" y="137.922" size="1.016" layer="96" font="vector" ratio="20" align="center-left"/>
-</instance>
-<instance part="SUPPLY1" gate="G$1" x="15.24" y="137.16" smashed="yes">
-<attribute name="VALUE" x="15.24" y="139.954" size="1.016" layer="96" font="vector" ratio="20" align="bottom-center"/>
-</instance>
-<instance part="C2" gate="G$1" x="15.24" y="111.76" smashed="yes">
-<attribute name="NAME" x="12.954" y="114.681" size="1.016" layer="95" font="vector" ratio="20"/>
-<attribute name="VALUE" x="11.176" y="110.871" size="1.016" layer="96" font="vector" ratio="20"/>
-</instance>
 <instance part="R2" gate="G$1" x="40.64" y="76.2" smashed="yes">
 <attribute name="NAME" x="36.83" y="76.454" size="1.016" layer="95" font="vector" ratio="20" align="bottom-center"/>
@@
 <nets>
 <net name="GND" class="0">
-<segment>
-<pinref part="GND" gate="1" pin="GND"/>
-<pinref part="C2" gate="G$1" pin="2"/>
-<wire x1="15.24" y1="109.22" x2="15.24" y2="101.6" width="0.1524" layer="91"/>
-<wire x1="15.24" y1="101.6" x2="15.24" y2="88.9" width="0.1524" layer="91"/>
-<wire x1="27.94" y1="101.6" x2="15.24" y2="101.6" width="0.1524" layer="91"/>
-<junction x="15.24" y="101.6"/>
-<pinref part="IC1" gate="G$1" pin="GND"/>
-<wire x1="38.1" y1="116.84" x2="27.94" y2="116.84" width="0.1524" layer="91"/>
-<wire x1="27.94" y1="116.84" x2="27.94" y2="101.6" width="0.1524" layer="91"/>
-</segment>
 <segment>
 <pinref part="D1" gate="G$1" pin="C"/>
@@
 <net name="SCL" class="0">
 <segment>
-<pinref part="IC1" gate="G$1" pin="DIO4"/>
-<wire x1="38.1" y1="129.54" x2="30.48" y2="129.54" width="0.1524" layer="91"/>
-<label x="30.48" y="129.54" size="1.016" layer="95" font="vector" ratio="20" rot="R180" xref="yes"/>
-</segment>
-<segment>
 <pinref part="J3" gate="G$1" pin="4"/>
 <wire x1="177.8" y1="58.42" x2="182.88" y2="58.42" width="0.1524" layer="91"/>
@@
 </net>
 <net name="VIN" class="0">
-<segment>
-<pinref part="IC1" gate="G$1" pin="VIN"/>
-<wire x1="38.1" y1="124.46" x2="15.24" y2="124.46" width="0.1524" layer="91"/>
-<pinref part="SUPPLY1" gate="G$1" pin="VIN"/>
-<wire x1="15.24" y1="137.16" x2="15.24" y2="124.46" width="0.1524" layer="91"/>
-<pinref part="C2" gate="G$1" pin="1"/>
-<wire x1="15.24" y1="116.84" x2="15.24" y2="124.46" width="0.1524" layer="91"/>
-<junction x="15.24" y="124.46"/>
-</segment>
 <segment>
 <pinref part="J3" gate="G$1" pin="2"/>
@@
 <net name="SDA" class="0">
 <segment>
-<pinref part="IC1" gate="G$1" pin="DIO5"/>
-<wire x1="38.1" y1="127" x2="30.48" y2="127" width="0.1524" layer="91"/>
-<label x="30.48" y="127" size="1.016" layer="95" font="vector" ratio="20" rot="R180" xref="yes"/>
-</segment>
-<segment>
 <pinref part="J3" gate="G$1" pin="3"/>
 <wire x1="177.8" y1="55.88" x2="182.88" y2="55.88" width="0.1524" layer="91"/>
@@
 <net name="TEST" class="0">
 <segment>
-<pinref part="IC1" gate="G$1" pin="ANATEST0/DIO14"/>
-<wire x1="38.1" y1="121.92" x2="33.02" y2="121.92" width="0.1524" layer="91"/>
-<label x="33.02" y="121.92" size="1.016" layer="95" font="vector" ratio="20" rot="R180" xref="yes"/>
-</segment>
-<segment>
 <pinref part="R2" gate="G$1" pin="1"/>
 <wire x1="35.56" y1="76.2" x2="27.94" y2="76.2" width="0.1524" layer="91"/>
 <label x="27.94" y="76.2" size="1.016" layer="95" font="vector" ratio="20" rot="R180" xref="yes"/>
 </segment>
+<segment>
+<pinref part="U3" gate="G$1" pin="P0.30"/>
+<wire x1="-63.5" y1="124.46" x2="-58.42" y2="124.46" width="0.1524" layer="91"/>
+<label x="-58.42" y="124.46" size="1.016" layer="95" font="vector" ratio="20" xref="yes"/>
+</segment>
 </net>
 <net name="N$1" class="0">
@@
 <net name="SWCLK" class="0">
 <segment>
-<pinref part="IC1" gate="G$1" pin="DIO9"/>
-<wire x1="83.82" y1="132.08" x2="91.44" y2="132.08" width="0.1524" layer="91"/>
-<label x="91.44" y="132.08" size="1.016" layer="95" font="vector" ratio="20" xref="yes"/>
-</segment>
-<segment>
 <pinref part="J1" gate="G$1" pin="SWDCLK/TCK"/>
 <wire x1="68.58" y1="38.1" x2="73.66" y2="38.1" width="0.1524" layer="91"/>
@@
 <net name="SWDIO" class="0">
 <segment>
-<pinref part="IC1" gate="G$1" pin="DIO10"/>
-<wire x1="83.82" y1="129.54" x2="91.44" y2="129.54" width="0.1524" layer="91"/>
-<label x="91.44" y="129.54" size="1.016" layer="95" font="vector" ratio="20" xref="yes"/>
-</segment>
-<segment>
 <pinref part="J1" gate="G$1" pin="SWDIO/TMS"/>
 <wire x1="68.58" y1="40.64" x2="73.66" y2="40.64" width="0.1524" layer="91"/>
@@
 <net name="TX" class="0">
 <segment>
-<pinref part="IC1" gate="G$1" pin="DIO8"/>
-<wire x1="38.1" y1="111.76" x2="33.02" y2="111.76" width="0.1524" layer="91"/>
-<label x="33.02" y="111.76" size="1.016" layer="95" font="vector" ratio="20" rot="R180" xref="yes"/>
-</segment>
-<segment>
 <pinref part="J4" gate="G$1" pin="VCC"/>
 <wire x1="101.6" y1="30.48" x2="111.76" y2="30.48" width="0.1524" layer="91"/>
@@
 <net name="RX" class="0">
 <segment>
-<pinref part="IC1" gate="G$1" pin="DIO11"/>
-<wire x1="83.82" y1="134.62" x2="91.44" y2="134.62" width="0.1524" layer="91"/>
-<label x="91.44" y="134.62" size="1.016" layer="95" font="vector" ratio="20" xref="yes"/>
-</segment>
-<segment>
 <pinref part="J4" gate="G$1" pin="SCL"/>
 <wire x1="101.6" y1="33.02" x2="111.76" y2="33.02" width="0.1524" layer="91"/>
@@
 <net name="NRST" class="0">
 <segment>
-<pinref part="IC1" gate="G$1" pin="RESETN"/>
-<wire x1="83.82" y1="114.3" x2="88.9" y2="114.3" width="0.1524" layer="91"/>
-<label x="88.9" y="114.3" size="1.016" layer="95" font="vector" ratio="20" xref="yes"/>
-</segment>
-<segment>
 <pinref part="J1" gate="G$1" pin="!RESET"/>
 <wire x1="68.58" y1="30.48" x2="73.66" y2="30.48" width="0.1524" layer="91"/>
@@
 </segment>
 <segment>
-<pinref part="IC1" gate="G$1" pin="DIO1"/>
-<wire x1="83.82" y1="116.84" x2="88.9" y2="116.84" width="0.1524" layer="91"/>
-<label x="88.9" y="116.84" size="1.016" layer="95" font="vector" ratio="20" xref="yes"/>
+<pinref part="U3" gate="G$1" pin="P1.08"/>
+<wire x1="-63.5" y1="99.06" x2="-55.88" y2="99.06" width="0.1524" layer="91"/>
+<label x="-55.88" y="99.06" size="1.016" layer="95" font="vector" ratio="20" xref="yes"/>
 </segment>
 </net>
@@
 </segment>
 <segment>
-<pinref part="IC1" gate="G$1" pin="DIO3"/>
-<wire x1="83.82" y1="119.38" x2="88.9" y2="119.38" width="0.1524" layer="91"/>
-<label x="88.9" y="119.38" size="1.016" layer="95" font="vector" ratio="20" xref="yes"/>
+<pinref part="U3" gate="G$1" pin="P0.13/IO0"/>
+<wire x1="-114.3" y1="81.28" x2="-119.38" y2="81.28" width="0.1524" layer="91"/>
+<label x="-119.38" y="81.28" size="1.016" layer="95" font="vector" ratio="20" rot="R180" xref="yes"/>
 </segment>
 </net>
@@
 </segment>
 <segment>
-<pinref part="IC1" gate="G$1" pin="DIO7/BOOT"/>
-<wire x1="38.1" y1="119.38" x2="33.02" y2="119.38" width="0.1524" layer="91"/>
-<label x="33.02" y="119.38" size="1.016" layer="95" font="vector" ratio="20" rot="R180" xref="yes"/>
-</segment>
-</net>
+<pinref part="U3" gate="G$1" pin="P1.15"/>
+<wire x1="-63.5" y1="81.28" x2="-58.42" y2="81.28" width="0.1524" layer="91"/>
+<label x="-58.42" y="81.28" size="1.016" layer="95" font="vector" ratio="20" xref="yes"/>
+</segment>
+</net>

Commit message: Update BT40_v23.sch
Changed lines of the file:
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@@
 <part name="GND11" library="Adafruit nRF52 Bluefruit Feather rev G" deviceset="SUPPLY1_GND" device="" value="GND"/>
 <part name="SUPPLY8" library="SparkFun-PowerSymbols" library_urn="urn:adsk.eagle:library:530" deviceset="3.3V" device=""/>
+<part name="FRAME2" library="SparkFun-Aesthetics" library_urn="urn:adsk.eagle:library:507" deviceset="FRAME-A4L" device=""/>
 </parts>
 <sheets>
@@
 </nets>
 </sheet>
+<sheet>
+<plain>
+</plain>
+<instances>
+<instance part="FRAME2" gate="G$1" x="0" y="0" smashed="yes">
+<attribute name="DRAWING_NAME" x="181.61" y="11.43" size="2.54" layer="94" font="vector"/>
+<attribute name="LAST_DATE_TIME" x="181.61" y="6.35" size="2.286" layer="94" font="vector"/>
+<attribute name="SHEET" x="195.58" y="1.27" size="2.54" layer="94" font="vector"/>
+</instance>
+</instances>
+<busses>
+</busses>
+<nets>
+</nets>
+</sheet>

Commit message: Update to design files
Parts:
- added R4: 0, SparkFun-Resistors:0OHM-0603-1/10W-5%
Connections:
- net 3.3V: now also R4.1
- net VIN: now also R4.2
Other:
- moved on the sheet: C4, U3
