File: hardware/v3/BT40_v23.brd (EAGLE design)
At the start: 74.3 x 73.2 mm, 14 parts, among them IC1 BLUENRG-M2SP, J1 CORTEX_DEBUG_SMD, J3 QWIIC, SW1 REVERSE_SWITCH, U1 BME680, U2 LSM6DSO32TRLGA-14L_2P5X3X0P83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

Commit message: Changes to design files
Parts:
- added U3: BT40F, BT40F:XCVR_BT40F
Connections:
- new net N$2: U3.15
- new net VBUS: U3.F6
- new net VDD: U3.9
- new net VDDH: U3.F4
- net GND: now also U3.10, U3.A0, U3.B0, U3.C0, U3.D0, U3.H0, U3.H1, U3.H2, U3.H3
Changed lines of the file:
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@@
 </element>
 <element name="SW1" library="reverse_mount_sw" package="REVERSE_TACTILE" value="REVERSE_SWITCH" x="-12.1412" y="-3.7592" smashed="yes"/>
+<element name="U3" library="BT40F" package="XCVR_BT40F" value="BT40F" x="-63.5" y="-39.37" smashed="yes">
+<attribute name="AVAILABILITY" value="In Stock" x="-63.5" y="-39.37" size="1.778" layer="27" display="off"/>
+<attribute name="DESCRIPTION" value=" 802.15.4, Bluetooth Bluetooth v5.1, Zigbee® Transceiver Module 2.4GHz PCB Trace Surface Mount " x="-63.5" y="-39.37" size="1.778" layer="27" display="off"/>
+<attribute name="MF" value="Fanstel Corp." x="-63.5" y="-39.37" size="1.778" layer="27" display="off"/>
+<attribute name="MP" value="BT40F" x="-63.5" y="-39.37" size="1.778" layer="27" display="off"/>
+<attribute name="NAME" x="-71" y="-27.87" size="1.27" layer="25"/>
+<attribute name="PACKAGE" value="SMD-66 Fanstel Corp." x="-63.5" y="-39.37" size="1.778" layer="27" display="off"/>
+<attribute name="PRICE" value="None" x="-63.5" y="-39.37" size="1.778" layer="27" display="off"/>
+<attribute name="PURCHASE-URL" value="https://pricing.snapeda.com/search/part/BT40F/?ref=eda" x="-63.5" y="-39.37" size="1.778" layer="27" display="off"/>
+<attribute name="VALUE" x="-71" y="-51.87" size="1.27" layer="27"/>
+</element>
 </elements>
 <signals>
@@
 <via x="3.7084" y="13.4112" extent="1-16" drill="0.381"/>
 <via x="7.4168" y="13.6906" extent="1-16" drill="0.381"/>
+<contactref element="U3" pad="H0"/>
+<contactref element="U3" pad="H3"/>
+<contactref element="U3" pad="H2"/>
+<contactref element="U3" pad="H1"/>
+<contactref element="U3" pad="10"/>
+<contactref element="U3" pad="B0"/>
+<contactref element="U3" pad="D0"/>
+<contactref element="U3" pad="C0"/>
+<contactref element="U3" pad="A0"/>
+<wire x1="-64.125" y1="-39.87" x2="-66.375" y2="-39.87" width="0" layer="19" extent="1-1"/>
+<wire x1="-63.75" y1="-41.87" x2="-64.125" y2="-39.87" width="0" layer="19" extent="1-1"/>
+<wire x1="-65.25" y1="-41.87" x2="-63.75" y2="-41.87" width="0" layer="19" extent="1-1"/>
+<wire x1="-62.25" y1="-41.87" x2="-63.75" y2="-41.87" width="0" layer="19" extent="1-1"/>
+<wire x1="-60.75" y1="-41.87" x2="-62.25" y2="-41.87" width="0" layer="19" extent="1-1"/>
+<wire x1="-61.875" y1="-39.87" x2="-62.25" y2="-41.87" width="0" layer="19" extent="1-1"/>
+<wire x1="-59.625" y1="-39.87" x2="-61.875" y2="-39.87" width="0" layer="19" extent="1-1"/>
+<wire x1="-56" y1="-47.67" x2="-60.75" y2="-41.87" width="0" layer="19" extent="1-1"/>
+<wire x1="-16.51" y1="-16.51" x2="-59.625" y2="-39.87" width="0" layer="19" extent="1-1"/>
+<wire x1="-14.1986" y1="-13.2334" x2="-16.51" y2="-16.51" width="0" layer="19" extent="1-1"/>
+<wire x1="-14.1986" y1="-11.9634" x2="-14.1986" y2="-13.2334" width="0" layer="19" extent="1-1"/>
+<wire x1="-17.1412" y1="-6.0092" x2="-14.1986" y2="-11.9634" width="0" layer="19" extent="1-1"/>
+<wire x1="-11.8172" y1="1.1676" x2="-17.1412" y2="-6.0092" width="0" layer="19" extent="1-1"/>
+<wire x1="-11.8172" y1="2.7876" x2="-11.8172" y2="1.1676" width="0" layer="19" extent="1-1"/>
+<wire x1="-9.4172" y1="3.5876" x2="-11.8172" y2="2.7876" width="0" layer="19" extent="1-1"/>
+<wire x1="-14.4018" y1="5.2696" x2="-11.8172" y2="2.7876" width="0" layer="19" extent="1-1"/>
+<wire x1="-9.1066" y1="11.9634" x2="-9.4172" y2="3.5876" width="0" layer="19" extent="1-1"/>
+<wire x1="-5.1622" y1="11.4238" x2="-9.1066" y2="11.9634" width="0" layer="19" extent="1-1"/>
+<wire x1="-0.8622" y1="13.9488" x2="-5.1622" y2="11.4238" width="0" layer="19" extent="1-1"/>
+<wire x1="1.3716" y1="13.8684" x2="-0.8622" y2="13.9488" width="0" layer="19" extent="1-1"/>
+<wire x1="3.7084" y1="13.4112" x2="1.3716" y2="13.8684" width="0" layer="19" extent="1-1"/>
+<wire x1="0.4378" y1="11.4238" x2="1.3716" y2="13.8684" width="0" layer="19" extent="1-1"/>
+<wire x1="1.0668" y1="16.9418" x2="1.3716" y2="13.8684" width="0" layer="19" extent="1-1"/>
+<wire x1="7.4168" y1="13.6906" x2="3.7084" y2="13.4112" width="0" layer="19" extent="1-1"/>
+<wire x1="-11.303" y1="17.2602" x2="-9.1066" y2="11.9634" width="0" layer="19" extent="1-1"/>
+<wire x1="-4.7566" y1="19.1422" x2="1.0668" y2="16.9418" width="0" layer="19" extent="1-1"/>
+<wire x1="-7.1412" y1="-6.0092" x2="-11.8172" y2="1.1676" width="0" layer="19" extent="1-1"/>
+<wire x1="5.9944" y1="3.3274" x2="0.4378" y2="11.4238" width="0" layer="19" extent="1-1"/>
+<wire x1="9.0424" y1="1.6345" x2="7.8321" y2="3.3408" width="0" layer="19" extent="1-1"/>
+<wire x1="12.4206" y1="0.1406" x2="9.5424" y2="1.6345" width="0" layer="19" extent="1-1"/>
+<wire x1="2.286" y1="-0.3086" x2="5.9944" y2="3.3274" width="0" layer="19" extent="1-1"/>
+<wire x1="16.51" y1="-15.24" x2="12.4206" y2="0.1406" width="0" layer="19" extent="1-1"/>
 </signal>
 <signal name="SCL">
@@
 <wire x1="-6.3754" y1="9.9568" x2="-6.3754" y2="17.2466" width="0.254" layer="1"/>
 </signal>
+<signal name="VDD">
+<contactref element="U3" pad="9"/>
+</signal>
+<signal name="VDDH">
+<contactref element="U3" pad="F4"/>
+</signal>
+<signal name="VBUS">
+<contactref element="U3" pad="F6"/>
+</signal>
+<signal name="N$2">
+<contactref element="U3" pad="15"/>
+</signal>
 </signals>

Commit message: Check-in
Connections:
- removed net N$2: U3.15
- net SWCLK: now also U3.15
Changed lines of the file:
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@@
 <wire x1="-11.5062" y1="7.747" x2="-14.5542" y2="7.747" width="0.254" layer="16"/>
 <wire x1="-14.5542" y1="7.747" x2="-15.2654" y2="7.0358" width="0.254" layer="16"/>
+<contactref element="U3" pad="15"/>
+<wire x1="-20.4216" y1="-12.9794" x2="-56" y2="-42.17" width="0" layer="19" extent="1-1"/>
 </signal>
 <signal name="SWDIO">
@@
 <contactref element="U3" pad="F6"/>
 </signal>
-<signal name="N$2">
-<contactref element="U3" pad="15"/>
-</signal>
 </signals>

Commit message: Changes
Parts:
- added C4: 0.1uF, SparkFun-Capacitors:0603
Connections:
- removed net VDDH: U3.F4
- net GND: now also C4.2
- net NRST: now also U3.14
- net SWDIO: now also U3.16
- net VIN: now also C4.1, U3.F4
Changed lines of the file:
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@@
 </layers>
 <board>
-<fusionsync huburn="a.cGVyc29uYWw6dWUyYWE1ODAx" projecturn="a.cGVyc29uYWw6dWUyYWE1ODAxIzIwMjIwNDE5NTE4MTIwODAx" f3durn="urn:adsk.wipprod:dm.lineage:abtfwLkORDeIlyAn2Un3pQ" pcbguid="" lastpulledtime="2022-04-19T18:14:00Z" lastsyncedchangeguid="" latestrevisionid="860d09df-7141-4c96-8803-181b72bb6630" lastsyncedrevisionid="860d09df-7141-4c96-8803-181b72bb6630" lastboardhashguid="" lastpushedtime="" linktopcb3d="true"/>
+<fusionsync huburn="a.cGVyc29uYWw6dWUyYWE1ODAx" projecturn="a.cGVyc29uYWw6dWUyYWE1ODAxIzIwMjIwNDE5NTE4MTIwODAx" f3durn="urn:adsk.wipprod:dm.lineage:abtfwLkORDeIlyAn2Un3pQ" pcbguid="" lastpulledtime="2022-04-19T18:14:00Z" lastsyncedchangeguid="" latestrevisionid="860d09df-7141-4c96-8803-181b72bb6630" lastsyncedrevisionid="860d09df-7141-4c96-8803-181b72bb6630" lastboardhashguid="" lastpushedtime="" linktopcb3d="false"/>
 <plain>
 <wire x1="10.7514" y1="-9.1438" x2="13.3708" y2="-14.0121" width="0.1524" layer="20"/>
@@
 <attribute name="VALUE" x="-71" y="-51.87" size="1.27" layer="27"/>
 </element>
+<element name="C4" library="SparkFun-Capacitors" library_urn="urn:adsk.eagle:library:510" package="0603" package3d_urn="urn:adsk.eagle:package:37414/1" value="0.1uF" x="-68.58" y="-55.88" smashed="yes">
+<attribute name="NAME" x="-68.58" y="-55.118" size="0.6096" layer="25" font="vector" ratio="20" align="bottom-center"/>
+<attribute name="PROD_ID" value="CAP-00810" x="-68.58" y="-55.88" size="1.778" layer="27" display="off"/>
+<attribute name="VALUE" x="-68.58" y="-56.642" size="0.6096" layer="27" font="vector" ratio="20" align="top-center"/>
+</element>
 </elements>
 <signals>
@@
 <contactref element="U3" pad="C0"/>
 <contactref element="U3" pad="A0"/>
-<wire x1="-64.125" y1="-39.87" x2="-66.375" y2="-39.87" width="0" layer="19" extent="1-1"/>
-<wire x1="-63.75" y1="-41.87" x2="-64.125" y2="-39.87" width="0" layer="19" extent="1-1"/>
-<wire x1="-65.25" y1="-41.87" x2="-63.75" y2="-41.87" width="0" layer="19" extent="1-1"/>
+<contactref element="C4" pad="2"/>
+<wire x1="-65.25" y1="-41.87" x2="-67.73" y2="-55.88" width="0" layer="19" extent="1-1"/>
+<wire x1="-63.75" y1="-41.87" x2="-65.25" y2="-41.87" width="0" layer="19" extent="1-1"/>
 <wire x1="-62.25" y1="-41.87" x2="-63.75" y2="-41.87" width="0" layer="19" extent="1-1"/>
 <wire x1="-60.75" y1="-41.87" x2="-62.25" y2="-41.87" width="0" layer="19" extent="1-1"/>
+<wire x1="-64.125" y1="-39.87" x2="-63.75" y2="-41.87" width="0" layer="19" extent="1-1"/>
 <wire x1="-61.875" y1="-39.87" x2="-62.25" y2="-41.87" width="0" layer="19" extent="1-1"/>
+<wire x1="-66.375" y1="-39.87" x2="-64.125" y2="-39.87" width="0" layer="19" extent="1-1"/>
 <wire x1="-59.625" y1="-39.87" x2="-61.875" y2="-39.87" width="0" layer="19" extent="1-1"/>
 <wire x1="-56" y1="-47.67" x2="-60.75" y2="-41.87" width="0" layer="19" extent="1-1"/>
@@
 <wire x1="-9.652" y1="-1.3208" x2="-10.2108" y2="-0.762" width="0.254" layer="16"/>
 <wire x1="-14.3002" y1="-0.254" x2="-14.3002" y2="0.508" width="0.254" layer="16"/>
+<contactref element="C4" pad="1"/>
+<contactref element="U3" pad="F4"/>
+<wire x1="-57.75" y1="-46.67" x2="-69.43" y2="-55.88" width="0" layer="19" extent="1-1"/>
+<wire x1="-14.1986" y1="-14.5034" x2="-57.75" y2="-46.67" width="0" layer="19" extent="1-1"/>
 </signal>
 <signal name="SDA">
@@
 <wire x1="-14.9606" y1="-5.334" x2="-18.7452" y2="-9.1186" width="0.254" layer="16"/>
 <wire x1="-18.7452" y1="-9.1186" x2="-18.7452" y2="-13.1318" width="0.254" layer="16"/>
+<contactref element="U3" pad="16"/>
+<wire x1="-19.0246" y1="-14.5034" x2="-56" y2="-41.07" width="0" layer="19" extent="1-1"/>
 </signal>
 <signal name="TX">
@@
 <wire x1="-16.4338" y1="-7.9502" x2="-16.8148" y2="-8.3312" width="0.254" layer="16"/>
 <wire x1="-16.8148" y1="-8.3312" x2="-16.8148" y2="-8.7122" width="0.254" layer="16"/>
+<contactref element="U3" pad="14"/>
+<wire x1="-19.0246" y1="-9.4234" x2="-56" y2="-43.27" width="0" layer="19" extent="1-1"/>
 </signal>
 <signal name="INT1">
@@
 <wire x1="-6.3754" y1="9.9568" x2="-6.3754" y2="17.2466" width="0.254" layer="1"/>
 </signal>
+<signal name="VBUS">
+<contactref element="U3" pad="F6"/>
+</signal>
 <signal name="VDD">
 <contactref element="U3" pad="9"/>
 </signal>
-<signal name="VDDH">
-<contactref element="U3" pad="F4"/>
-</signal>
-<signal name="VBUS">
-<contactref element="U3" pad="F6"/>
-</signal>
 </signals>

Commit message: Update to schematic
Parts:
- moved U3 29.3 mm to (-54.6, -11.4)
Connections:
- net VDD renamed 3.3V
- new net SWO: J1.6, U3.12
- net GND: now also J1.9
- net RX: now also U3.D5
- net SCL: now also U3.2
- net SDA: now also U3.1
- net TX: now also U3.C5

Commit message: Check-in
Parts:
- removed C2: 0.1uF, SparkFun-Capacitors:0603
- removed IC1: BLUENRG-M2SP, SamacSys_Parts:BLUENRGM2SP
Connections:
- net BUTTON: now also U3.Z6; no longer IC1.7
- net GND: no longer C2.2, IC1.8
- net INT1: now also U3.A6; no longer IC1.18
- net INT2: now also U3.B6; no longer IC1.17
- net NRST: no longer IC1.19
- net RX: no longer IC1.11
- net SCL: no longer IC1.3
- net SDA: no longer IC1.4
- net SWCLK: no longer IC1.12
- net SWDIO: no longer IC1.13
- net TEST: now also U3.13; no longer IC1.6
- net TX: no longer IC1.10
- net VIN: no longer C2.1, IC1.5
Routing:
- net VIN: track 125.4 -> 121.8 mm
- net SWCLK: track 57.5 -> 54.7 mm
- net TX: track 29.6 -> 28.0 mm
- net NRST: track 65.0 -> 63.6 mm
- net SDA: track 52.6 -> 51.3 mm
- net INT1: track 34.0 -> 32.7 mm
- net SCL: track 53.1 -> 51.9 mm

Commit message: Update to design files
Parts:
- added R4: 0, SparkFun-Resistors:0603
- moved C4 100.8 mm to (3.78, 14.2)
- moved U3 64.7 mm to (-2.21, 26.5)
- moved R2 1.75 mm to (-8.18, 14.0), turned to 0 degrees
Connections:
- net 3.3V: now also R4.1
- net VIN: now also R4.2
Routing:
- net NRST: track 63.6 -> 0.00 mm, vias 7 -> 0
- net SWDIO: track 58.7 -> 0.00 mm, vias 2 -> 0
- net SWCLK: track 54.7 -> 0.00 mm, vias 2 -> 0
- net VIN: track 121.8 -> 69.7 mm, vias 8 -> 0
- net SCL: track 51.9 -> 0.00 mm, vias 2 -> 0
- net SDA: track 51.3 -> 0.00 mm, vias 5 -> 0
- net BUTTON: track 39.8 -> 0.00 mm
- net INT1: track 32.7 -> 0.00 mm, vias 2 -> 0
- net TX: track 28.0 -> 0.00 mm, vias 2 -> 0
- net INT2: track 25.8 -> 0.00 mm, vias 2 -> 0
- net RX: track 20.6 -> 0.00 mm, vias 2 -> 0
- net GND: track 4.15 -> 0.00 mm, vias 6 -> 0
- net N$1: track 2.75 -> 0.00 mm
- net TEST: track 2.73 -> 0.00 mm

Commit message: Completed PCB design
Parts:
- moved R1 1.43 mm to (-2.74, 6.88)
- moved R3 1.40 mm to (-4.50, 6.93)
Routing:
- net NRST: track 0.00 -> 71.6 mm, vias 0 -> 2
- net SWDIO: track 0.00 -> 60.1 mm, vias 0 -> 2
- net SWCLK: track 0.00 -> 59.6 mm, vias 0 -> 2
- net SWO: track 0.00 -> 58.7 mm, vias 0 -> 2
- net SCL: track 0.00 -> 54.7 mm, vias 0 -> 7
- net SDA: track 0.00 -> 51.1 mm, vias 0 -> 5
- net INT1: track 0.00 -> 45.5 mm, vias 0 -> 2
- net VIN: track 69.7 -> 112.9 mm, vias 0 -> 4
- net RX: track 0.00 -> 41.8 mm, vias 0 -> 4
- net INT2: track 0.00 -> 36.6 mm, vias 0 -> 4
- net TX: track 0.00 -> 34.5 mm, vias 0 -> 4
- net BUTTON: track 0.00 -> 31.8 mm, vias 0 -> 2
- net TEST: track 0.00 -> 28.9 mm, vias 0 -> 2
- net GND: track 0.00 -> 5.13 mm, vias 0 -> 7
- net 3.3V: track 0.00 -> 2.54 mm
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